File: projects/onboard_flight_computer/obc.sch (EAGLE design)
At the start: 228 parts, among them IC1 IS42S16160J-6BLI, IC2 S26KS512SDPBHI020, IC3 74LVC2T45GS,115, IC4 74LVCH1T45GS,132, IC5 MIMXRT1052DVJ6B, IC7 74LVCH1T45GS,132, IC8 74LVCH1T45GS,132, J1 504050-0791, J2 DX4R205JJAR1800, J3 504050-0791, J4 504050-0791, J5 504050-0791, J6 ESQ-126-37-G-D, J7 FH28-10S-0.5SH_05_, J8 504050-1091, J9 ESQ-126-37-G-D, Q1 FA-128, Q3 FC-12M, U10 HONEYWELL_HMC5983-TRHONEYWELL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, U11 HONEYWELL_HMC5983-TRHONEYWELL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, U12 HONEYWELL_HMC5983-TRHONEYWELL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, U13 DS1307N, U2 MCP1702T-1802E/CB, U3 NXP_FXAS21002CQR1NXP_FXAS2100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, U4 MK20DX128VFM5, U5 NLX2G14CMUTCG, U6 NTSX2102GU8H, U7 NXP_FXAS21002CQR1NXP_FXAS2100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, U8 NX5P3090UKZ, U9 NXP_FXAS21002CQR1NXP_FXAS2100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, Y1 ECS-.327-12.5-13X

Commit message: Update obc.sch
Parts:
- removed BT1: BA2032SM, BA2032SM:BA2032SM
- removed C65, C69, C82: 10 uF, rcl:C-EUC0402K
- removed C66: 2.2 uF, rcl:C-EUC0402K
- removed C67, C72, C73, C76, C77, C78, C81, C85, C88, C89, C92, C93, C96: 0.1 uF, rcl:C-EUC0402K
- removed C68, C86, C90, C94: 1.0 uF, rcl:C-EUC0402K
- removed C70, C71: 22 pF, rcl:C-EUC0402K
- removed C74, C80, C83: 4.7 uF, rcl:C-EUC0402K
- removed C75, C84: 0.22 uF, rcl:C-EUC0402K
- removed C79: 1000 pF, rcl:C-EUC0402K
- removed C87, C91, C95: 100 nF, rcl:C-EUC0402K
- removed D10, D8, D9: 0402ESDA-MLP1, 0402ESDA-MLP1:0402ESDA-MLP1
- removed D5: KINGBRIGHT_KPT-1608SGCKINGBRIGHT_KPT-1608SGC_0_0, Kingbright - KPT-1608SGC:KINGBRIGHT_KPT-1608SGCKINGBRIGHT_KPT-1608SGC_0_0
- removed D6: RB521S30T1G, RB521S30T1G:RB521S30T1G
- removed FB2: MPZ1608S331A, MPZ1608S331A:MPZ1608S331A
- removed IC2: S26KS512SDPBHI020, SDRAM_and_HyperFlash:S26KS512SDPBHI020
- removed IC3: 74LVC2T45GS,115, 74LVC2T45GS_115:74LVC2T45GS,115
- removed IC4: 74LVCH1T45GS,132, 74LVCH1T45GS_132:74LVCH1T45GS,132
- removed IC5: MIMXRT1052DVJ6B, MIMXRT1052DVJ6B:MIMXRT1052DVJ6B
- removed J3, J4, J5: 504050-0791, 504050-0791:504050-0791
- removed J6, J9: ESQ-126-37-G-D, ESQ-126-37-G-D:ESQ-126-37-G-D
- removed J7: FH28-10S-0.5SH_05_, FH28-10S-0.5SH_05_:FH28-10S-0.5SH_05_
- removed J8: 504050-1091, 504050-1091:504050-1091
- removed JP1: 20, pinhead:PINHD-2X10
- removed L1: 120 Ohm, inductors:BLM15HB121SN1
- removed Q1: FA-128, crystal:FA-128
- removed Q3: FC-12M, crystal:FC-12M
- removed R100: 15k, ngspice-simulation:R
- removed R114, R134: 1k Ohm, rcl:R-EU_R0402
- removed R64, R82, R83, R84, R85, R88, R89, R91, R92, R94, R95, R98: 10k, ngspice-simulation:R
- removed R65, R81, R87, R90, R93: 4.7k, ngspice-simulation:R
- removed R74, R75: 33, ngspice-simulation:R
- removed R76: 0, ngspice-simulation:R
- removed R80: CSTCE8M00G55-R0, CSTCE8M00G55-R0:CSTCE8M00G55-R0
- removed R86: 180k, ngspice-simulation:R
- removed R96: 220, ngspice-simulation:R
- removed R97: 100k, ngspice-simulation:R
- removed R99: 1k, ngspice-simulation:R
- removed S1: TL3301AF260QG, TL3301AF260QG:TL3301AF260QG
- removed TP1, TP10, TP12, TP13, TP14, TP15, TP3: TPTP06R, testpad:TPTP06R
- removed U10, U11, U12: HONEYWELL_HMC5983-TRHONEYWELL_HMC5983-TR_0_0, Honeywell - HMC5983-TR:HONEYWELL_HMC5983-TRHONEYWELL_HMC5983-TR_0_0
- removed U13: DS1307N, DS1307N:DS1307N
- removed U2: MCP1702T-1802E/CB, MCP1702T1802ECB:MCP1702T-1802E/CB
- removed U3, U7, U9: NXP_FXAS21002CQR1NXP_FXAS21002CQR1_0_0, NXP - FXAS21002CQR1:NXP_FXAS21002CQR1NXP_FXAS21002CQR1_0_0
- removed U4: MK20DX128VFM5, MK20DX128VFM5:MK20DX128VFM5
- removed U5: NLX2G14CMUTCG, NLX2G14CMUTCG:NLX2G14CMUTCG
- removed U6: NTSX2102GU8H, NTSX2102GU8H:NTSX2102GU8H
- removed U8: NX5P3090UKZ, NX5P3090UKZ:NX5P3090UKZ
- added C4: 0.1uF, rcl:C-EUC0402K
- added D1, D3: BAT54XV2T1G, BAT54XV2T1G:BAT54XV2T1G
- added H1, H2: ESQ-126-39-G-D, ESQ-126-39-G-D:ESQ-126-39-G-D
- added IC10: IS25LP064A-JBLE, IS25LP064A-JBLE:IS25LP064A-JBLE
- added IC9: IS42S16160J-6TL, IS42S16160J-6TL:IS42S16160J-6TL
- added PS1: PJ-040D, PJ-040D:PJ-040D
- added R42, R45, R49, R51, R52, R53, R54, R55, R56, R57, R60, R61, R62: 0 Ohm, rcl:R-EU_R0402
- added TP5, TP8: TPTP06R, testpad:TPTP06R
- added Y2: ECS-.327-7-12-TR, ECS-.327-7-12-TR:ECS-.327-7-12-TR
- C14: value 0.22uF -> 10 uF
- C16, C19, C31, C33, C48: value 4.7uF -> 0.22uF
- C17, C23, C36: value 0.22uF -> 0.1uF
- C18, C24, C35: value 0.22uF -> 4.7uF
- C2, C51: value 0.1uF -> 4.7uF
- C3: value 4.7uF -> 1.0 uF
- C32, C43: value 10uF -> 0.1uF
- C37: value 33uF -> 0.1uF
- C39: value 4.7uF -> 4.7pF
- C40: value 0.22uF -> 4.7pF
- C41, C42: value 0.22uF -> 10pF
- C44, C45, C46, C47: value 0.1uF -> 0.22uF
- C5: value 22uF -> 1.0uF
- C50: value 0.1uF -> 1.0uF
- C52: value 4.7uF -> 1.0uF
- C53, C54, C55: value 4.7uF -> 0.1uF
- C57: value 0.1 uF -> 0.1uF
- C58: value 4.7 uF -> 0.1uF
- C59: value 0.22 uF -> 0.1uF
- C60, C61, C62: value 0.1 uF -> 4.7uF
- C63, C64: value 18pF -> 4.7uF
- D2: value RB521S30T1G -> BAT54XV2T1G; device RB521S30T1G:RB521S30T1G -> BAT54XV2T1G:BAT54XV2T1G
- D4: value KINGBRIGHT_KPT-1608SGCKINGBRIGHT_KPT-1608SGC_0_0 -> BAT54XV2T1G; device Kingbright - KPT-1608SGC:KINGBRIGHT_KPT-1608SGCKINGBRIGHT_KPT-1608SGC_0_0 -> BAT54XV2T1G:BAT54XV2T1G
- FB1: value MPZ1608S331A -> BLM15AG121SN1D; device MPZ1608S331A:MPZ1608S331A -> BLM15AG121SN1D:BLM15AG121SN1D
- IC1: value IS42S16160J-6BLI -> TPS3839L30DBZR; device SDRAM_and_HyperFlash:IS42S16160J-6BLI -> TPS3839L30DBZR:TPS3839L30DBZR
- IC7: value 74LVCH1T45GS,132 -> MIMXRT1021DAG5A; device 74LVCH1T45GS_132:74LVCH1T45GS,132 -> MIMXRT1021DAG5A:MIMXRT1021DAG5A
- IC8: value 74LVCH1T45GS,132 -> MIC94305YMT-TR; device 74LVCH1T45GS_132:74LVCH1T45GS,132 -> MIC94305YMT-TR:MIC94305YMT-TR
- J1: value 504050-0791 -> 504077-1891; device 504050-0791:504050-0791 -> 504077-1891:504077-1891
- J2: value DX4R205JJAR1800 -> 12214-8250-00FR; device DX4R205JJAR1800:DX4R205JJAR1800 -> 12214-8250-00FR:12214-8250-00FR
- L2: value 4.7 uH -> SRN4026-4R7M; device inductors:BLM15HB121SN1 -> SRN4026-4R7M:SRN4026-4R7M
- R1, R5, R59: value 0 Ohm -> 10k Ohm
- R10: value 2.2k -> 2.2M Ohm; device ngspice-simulation:R -> rcl:R-EU_R0402
- R11: value 2.2k -> 30k Ohm; device ngspice-simulation:R -> rcl:R-EU_R0402
- R12: value 2.2M Ohm -> 0 Ohm
- R14, R15: value 100K Ohm -> 0 Ohm
- R17, R18, R3: value 10k Ohm -> 0 Ohm
- R19, R28, R29, R30: value 2.2k -> 0 Ohm; device ngspice-simulation:R -> rcl:R-EU_R0402
- R26: value 10k Ohm -> 100 Ohm
- R31, R32, R33, R34, R35, R41: value 4.7k -> 0 Ohm; device ngspice-simulation:R -> rcl:R-EU_R0402
- R36, R37: value 4.7K Ohm -> 0 Ohm
- R46: value 10K Ohm -> 0 Ohm
- R6: value 30K Ohm -> 10k Ohm
- R8: value 4.7 k -> 0 Ohm; device rcl:R-US_R0805 -> rcl:R-EU_R0402
- R9: value 4.7k -> 1k Ohm; device rcl:R-US_R0805 -> rcl:R-EU_R0402
- Y1: value ECS-.327-12.5-13X -> XRCGB24M000F2P01R0; device ECS-.327-12.5-13X:ECS-.327-12.5-13X -> XRCGB24M000F2P01R0:XRCGB24M000F2P01R0
Connections:
- removed net 12V_BUS: J9.23, J9.24
- removed net 12V_PDM1: J9.8
- removed net 12V_PDM2: J9.10
- removed net 3V3_PDM10: J9.20
- removed net 3V3_PDM8: J9.18
- removed net 3V3_PDM9: C57.1, C60.1, C61.1, C62.1, C72.1, C73.1, C85.1, C86.1, C88.1, C89.1, C90.1, C92.1, C93.1, C94.1, C96.1, J7.6, J9.19, R10.1, R11.2, R19.1, R28.2, R29.1, R30.2, R31.2, R32.2, R33.2, R34.2, R35.2, R41.2, U10.!SPI_CS!(S1), U10.I2C/!SPI!, U10.VDD, U10.VDDIO, U11.!SPI_CS!(S1), U11.I2C/!SPI!, U11.VDD, U11.VDDIO, U12.!SPI_CS!(S1), U12.I2C/!SPI!, U12.VDD, U12.VDDIO, U3.SA0/MISO, U3.SPI_!CS!, U3.VDD, U3.VDDIO, U7.SA0/MISO, U7.SPI_!CS!, U7.VDD, U7.VDDIO, U9.SA0/MISO, U9.SPI_!CS!, U9.VDD, U9.VDDIO
- removed net 5V_BUS: J9.25, J9.26, R8.1, R9.1, U13.VCC
- removed net 5V_PDM5: J8.3, J9.13
- removed net 5V_PDM6: J1.1, J3.1, J4.1, J5.1, J9.15
- removed net 5V_PDM7: J8.1, J9.16
- removed net 5V_USB_CHARGE: D8.2, FB1.1, J2.1, J6.32
- removed net AAA: R100.2, R99.1, U8.EN
- removed net BATV_BUS: J9.45, J9.46
- removed net BATV_PDM3: J9.11
- removed net BATV_PDM4: J9.12
- removed net CAN_STBY: IC5.GPIO_AD_B0_05, R44.2
- removed net CHASSIS: J7.7, J9.50
- removed net DCDC_3V3: C1.1, C14.1, C15.1, C18.1, C19.1, C2.1, C3.1, D6.A, IC5.NVCC_EMC_1, IC5.NVCC_EMC_2, IC5.VDDA_ADC_3P3, IC5.VDD_HIGH_IN, L1.1, R1.2, R114.2, R134.2, R27.1, R63.2, R7.2
- removed net FLASH_RST: IC5.GPIO_B0_00, R2.1
- removed net FLASH_VCC: C51.1, C52.1, C55.1, C56.1, IC2.VCC, IC2.VCCQ_1, IC2.VCCQ_2, IC5.NVCC_SD1, R17.1, R18.1, R3.1, R4.2
- removed net FLEXSPI_CLK_B: IC2.CK#, IC5.GPIO_SD_B1_04
- removed net FLEXSPI_D0_B: IC2.DQ4, IC5.GPIO_SD_B1_03
- removed net FLEXSPI_D1_B: IC2.DQ5, IC5.GPIO_SD_B1_02
- removed net FLEXSPI_D2_B: IC2.DQ6, IC5.GPIO_SD_B1_01
- removed net FLEXSPI_D3_B: IC2.DQ7, IC5.GPIO_SD_B1_00
- removed net FLEXSPI_DQS: IC5.GPIO_SD_B1_05, R21.1
- removed net GPIO_AD_B1_00: IC5.GPIO_AD_B1_00, R58.2
- removed net GPIO_AD_B1_01: IC5.GPIO_AD_B1_01, R59.2
- removed net LDO_1V8: C49.1, C50.1, R4.1, TP3.TP, U2.VOUT
- removed net MCU_DCDC_IN: C39.1, C40.1, C41.1, C42.1, IC5.DCDC_IN_1, IC5.DCDC_IN_2, IC5.DCDC_IN_Q, R6.2, R7.1
- removed net N$27: IC2.INT#, R18.2
- removed net N$29: IC2.RESET#, R2.2
- removed net N$31: IC2.CS#, R20.2, R3.2
- removed net N$34: IC2.CK, R22.2
- removed net N$37: JP1.19, R26.2
- removed net N$39: D2.K, JP1.15
- removed net N$40: C32.1, C38.1, R1.1, U2.VIN
- removed net N$46: C75.1, U10.SETP
- removed net N$48: C59.1, U11.SETP
- removed net N$49: C84.2, U12.SETC
- removed net N$53: C63.2, IC5.RTC_XTALI, Q3.2
- removed net N$54: R81.1, U6.OE
- removed net N$56: C83.1, U12.C1
- removed net N$57: TP12.TP, U6.A2
- removed net N$60: TP13.TP, U6.B2
- removed net N$67: C91.1, U7.VREGD
- removed net N$71: C87.1, U3.VREGD
- removed net N$72: C95.1, U9.VREGD
- removed net N$76: D11.ANODE, R134.1
- removed net P3V3_SDA: C67.1, C68.1, C69.1, C76.1, C78.1, IC3.VCC(A), IC4.VCC(A), IC7.VCC(A), IC8.VCC(A), R76.1, R81.2, R82.2, R83.2, R85.2, R87.2, R90.2, R93.2, R96.2, R98.2, U4.VBAT, U4.VDD, U4.VDDA, U5.VCC, U6.VCCA
- removed net P5V_SDA: C65.1, C81.1, C82.1, FB1.2, R65.2, U4.VREGIN, U8.VINT
- removed net P5V_SDA_S: C80.1, U8.VBUS
- removed net PCM_IN: J9.35, J9.36
- removed net POWER_EN: R99.2, U4.PTD6/LLWU_P15
- removed net POWER_LED: D5.ANODE, R114.1
- removed net SDA_EXTAL: C70.1, R80.3, U4.PTA18
- removed net SDA_LED: D4.CATHODE, U4.PTD4/LLWU_P14
- removed net SDA_RST: R64.2, R65.1, TP7.TP, U4.RESET_B
- removed net SDA_RST_TGTMCU_B: C79.1, R40.1, R85.1, R86.1, S1.COM_2, S1.N.O._2, U4.PTB1, U6.A1, U6.B1
- removed net SDA_RX_EN: IC4.DIR, R87.1, R88.2
- removed net SDA_SPI0_CS: TP15.TP, U4.PTC2
- removed net SDA_SPI0_RST_B: TP14.TP, U4.PTC1/LLWU_P6
- removed net SDA_SPI0_SCK: IC8.A, U4.PTC5/LLWU_P9
- removed net SDA_SPI0_SIN: IC3.2A, U4.PTC7
- removed net SDA_SPI0_SOUT: IC7.A, U4.PTC6/LLWU_P10
- removed net SDA_SWD_EN: IC8.DIR, R93.1, R94.2, U5.OUT!Y1
- removed net SDA_SWD_EN_B: R83.1, U4.PTA4/LLWU_P3, U5.INA1
- removed net SDA_SWD_OE: IC7.DIR, R90.1, R91.2, U5.OUT!Y2
- removed net SDA_SWD_OE_B: R82.1, U4.PTB0/LLWU_P5, U5.INA2
- removed net SDA_USBSHIELD: FB2.2, J2.SHIELD
- removed net SDA_USB_CONN_DN: D10.2, J2.2, R75.1
- removed net SDA_USB_CONN_DP: D9.2, J2.3, R74.1
- removed net SDA_USB_DN: R75.2, U4.USB0_DM
- removed net SDA_USB_DP: R74.2, U4.USB0_DP
- removed net SDA_VOUT33: C66.1, R76.2, U4.VOUT33
- removed net SDA_XTAL: C71.1, R80.1, U4.PTA19
- removed net SPI1_EN_1: IC5.GPIO_B0_07, J1.2
- removed net SPI1_EN_2: IC5.GPIO_B0_08, J3.2
- removed net SPI1_EN_3: IC5.GPIO_B0_09, J4.2
- removed net SPI1_EN_4: IC5.GPIO_B0_10, J5.2
- removed net SPI1_NSS_1: J1.6, R43.1
- removed net SPI1_NSS_2: IC5.GPIO_AD_B0_04, J3.6
- removed net SPI1_NSS_3: J4.6, R44.1
- removed net SPI1_NSS_4: IC5.GPIO_AD_B0_14, J5.6
- removed net SWD_CLK: IC8.B, R48.1, R92.1
- removed net SWD_DIO: IC3.2B, IC7.B, R47.1, R89.1
- removed net TC_SDA_USB_ID_TP: J2.4, TP10.TP
- removed net UART1_RXD: IC4.B, IC5.GPIO_AD_B0_13, R84.1
- removed net UART1_RX_TGTMCU_R: IC4.A, U4.PTC4/LLWU_P8
- removed net UART1_TXD: IC3.1B, IC5.GPIO_AD_B0_12, R95.1
- removed net UART1_TX_TGTMCU_R: IC3.1A, U4.PTC3/LLWU_P7
- removed net UART2_RX: IC5.GPIO_AD_B1_03, J6.3
- removed net UART2_TX: IC5.GPIO_AD_B1_02, J6.1
- removed net UART8_RX: IC5.GPIO_AD_B1_11, J8.8
- removed net UART8_TX: IC5.GPIO_AD_B1_10, J8.7
- removed net USB_OTG1_ID: IC5.GPIO_AD_B0_01, R36.1, R39.2
- removed net USB_OTG1_OC: IC5.GPIO_AD_B0_03, R43.2
- removed net VDD_SOC_IN: C22.1, C23.1, C24.1, C25.1, C26.1, C27.1, C28.1, C29.1, C30.1, C31.1, IC5.DCDC_SENSE, IC5.VDD_SOC_IN_1, IC5.VDD_SOC_IN_2, IC5.VDD_SOC_IN_3, IC5.VDD_SOC_IN_4, R5.1
- removed net VTRG_FAULT_B: R98.1, U4.PTD7, U8.!FAULT
- removed net V_TGTMCU: C77.1, IC3.VCC(B), IC4.VCC(B), IC7.VCC(B), IC8.VCC(B), R84.2, R86.2, R89.2, R92.2, R95.2, U6.VCCB
- new net 5V_USB_OTG: C3.2, IC7.USB_OTG1_VBUS
- new net FLASH_3V3: C32.2, C5.2, IC10.VCC, R1.1, R4.2
- new net GPANAIO: IC7.GPANAIO, TP7.TP
- new net GPIO_EMC_16: IC9.A0, R49.1
- new net GPIO_EMC_17: IC9.A1, R50.1
- new net GPIO_EMC_18: IC9.A2, R51.1
- new net GPIO_EMC_19: IC9.A3, R52.1
- new net GPIO_EMC_20: IC9.A4, R32.2
- new net GPIO_EMC_21: IC9.A5, R31.2
- new net GPIO_EMC_22: IC9.A6, R30.2
- new net GPIO_EMC_23: IC9.A7, R29.2
- new net GPIO_EMC_24: IC9.A8, R28.2
- new net GPIO_EMC_25: IC9.A9, R25.2
- new net GPIO_EMC_26: IC9.A11, R24.2
- new net GPIO_EMC_27: IC9.A12, R23.2
- new net INT1_COMBO: IC7.GPIO_SD_B1_04, R7.1
- new net JTAG_DACK: J2.13, R26.1
- new net JTAG_NSRST: D2.K, J2.12
- new net N$12: IC9.DQ3, R39.1
- new net N$14: IC9.NC_4, R40.1
- new net N$15: J1.CLK, R56.2
- new net N$16: IC9.NC_5, R41.1
- new net N$17: IC9.!WE, R42.1
- new net N$18: IC9.!CAS, R43.1
- new net N$19: IC9.!RAS, R44.1
- new net N$20: IC9.!CS, R45.1
- new net N$21: IC9.BA0, R46.1
- new net N$22: IC9.BA1, R47.1
- new net N$23: IC9.A10, R48.1
- new net N$24: D3.A, D4.A, R60.1, R61.1
- new net N$25: J1.DAT0, R57.2
- new net N$42: IC9.DQ5, R16.2
- new net NVCC_PLL: C22.2, IC7.NVCC_PLL
- new net NVCC_SD0: C1.2, C2.2, IC7.NVCC_SD0, R3.2
- new net PMIC_STBY_REQ: IC7.PMIC_STBY_REQ, TP6.TP
- new net RTC_XTALI: C41.2, IC7.RTC_XTALI, Y2.IN/OUT
- new net SD1_CLK: IC7.GPIO_SD_B0_03, R56.1
- new net SD1_CMD: IC7.GPIO_SD_B0_02, R5.2, R55.1
- new net SD1_D0: IC7.GPIO_SD_B0_04, R57.1, R6.2
- new net SD1_D1: IC7.GPIO_SD_B0_05, R58.1
- new net SD1_D2: IC7.GPIO_SD_B0_00, R53.1
- new net SD1_D3: IC7.GPIO_SD_B0_01, R54.1
- new net SD_CD_SW: IC7.GPIO_SD_B0_06, J1.9, R59.1
- new net SD_PWREN: D3.K, R7.2
- new net SPI1_EN0: H1.9, IC7.GPIO_AD_B1_00
- new net SPI1_EN1: H1.10, IC7.GPIO_AD_B1_01
- new net SPI1_EN2: H1.22, IC7.GPIO_AD_B1_02
- new net SPI1_EN3: H1.21, IC7.GPIO_AD_B1_03
- new net SPI1_PCS0: H1.7, IC7.GPIO_AD_B0_11
- new net SPI1_PCS1: H1.8, IC7.GPIO_AD_B1_04
- new net SPI1_PCS2: H1.20, IC7.GPIO_AD_B1_05
- new net SPI1_PCS3: H1.19, IC7.GPIO_AD_B1_06
- new net UART1_RX: H1.4, IC7.GPIO_AD_B0_07
- new net UART1_TX: H1.2, IC7.GPIO_AD_B0_06
- new net UART4_RX: H1.3, IC7.GPIO_AD_B1_11
- new net UART4_TX: H1.1, IC7.GPIO_AD_B1_10
- new net USB_OTG1_CHD: IC7.USB_OTG1_CHD_B, TP5.TP
- new net VDD_HIGH_CAP: C23.2, C24.2, IC7.VDD_HIGH_CAP
- new net VDD_SNVS_CAP: C21.2, IC7.VDD_SNVS_CAP
- new net VSD_3V3: C38.2, C49.2, C52.2, IC8.VOUT, J1.VDD
- new net WAKEUP: IC7.WAKEUP, TP8.TP
- new net XTALO: C40.2, IC7.XTALO, Y1.XTAL_1
- net 3V3_BUS: now also C15.2, C16.2, C17.2, C18.2, C19.2, C37.2, C43.2, C47.2, C48.2, C50.2, C51.2, D1.A, D11.ANODE, FB1.1, H2.27, H2.28, IC7.DCDC_IN, IC7.DCDC_IN_Q, IC7.VDDA_ADC_3P3, IC7.VDD_HIGH_IN, IC8.VIN, J2.8, R11.2, R27.2, R3.1, R4.1, R5.1, R59.2, R6.1, R61.2, R62.2, R9.1; no longer IC5.NVCC_SD0, J9.27, J9.28
- net ANT_BURN_WIRE1: now also H1.23, IC7.GPIO_AD_B1_07; no longer IC5.GPIO_B0_11, J6.24
- net ANT_BURN_WIRE2: now also H1.25, IC7.GPIO_AD_B1_12; no longer IC5.GPIO_B0_13, J6.26
- net BCR_OUT: now also H2.41, H2.42, H2.43, H2.44, PS1.1; no longer J9.41, J9.42, J9.43, J9.44
- net DCDC_OUT: now also C25.2, C26.2, C27.2, C28.2, C29.2, C30.2, C31.2, C33.2, C34.2, C35.2, C45.2, C46.2, IC7.VDD_SOC_IN_1, IC7.VDD_SOC_IN_2, IC7.VDD_SOC_IN_3, IC7.VDD_SOC_IN_4, IC7.VDD_SOC_IN_5, IC7.VDD_SOC_IN_6, IC7.VDD_SOC_IN_7, L2.1; no longer C36.1, C37.1, L2.2, R5.2
- net DTR: now also H1.5, IC7.GPIO_SD_B1_05; no longer IC5.GPIO_B0_12, J8.6
- net FLEXSPI_CLK: now also IC10.SCK, IC7.GPIO_SD_B1_07; no longer IC5.GPIO_SD_B1_07, R22.1
- net FLEXSPI_D0_A: now also IC10.SI_(IO0), IC7.GPIO_SD_B1_08; no longer IC5.GPIO_SD_B1_08, R24.2
- net FLEXSPI_D1_A: now also IC10.SO_(IO1), IC7.GPIO_SD_B1_10; no longer IC5.GPIO_SD_B1_09, R23.2
- net FLEXSPI_D2_A: now also IC10.WP#_(IO2), IC7.GPIO_SD_B1_09; no longer IC5.GPIO_SD_B1_10, R16.2
- net FLEXSPI_D3_A: now also IC10.HOLD#_(IO3), IC7.GPIO_SD_B1_06; no longer IC5.GPIO_SD_B1_11, R25.2
- net FLEXSPI_SS0: now also IC10.CE#, IC7.GPIO_SD_B1_11, R1.2; no longer IC5.GPIO_SD_B1_06, R20.1
- net GND: now also C1.1, C14.1, C15.1, C16.1, C17.1, C18.1, C19.1, C2.1, C20.1, C21.1, C22.1, C23.1, C24.1, C25.1, C26.1, C27.1, C28.1, C29.1, C3.1, C30.1, C31.1, C32.1, C33.1, C34.1, C35.1, C36.1, C37.1, C38.1, C39.1, C4.1, C40.1, C41.1, C42.1, C43.1, C44.1, C45.1, C46.1, C47.1, C48.1, C49.1, C5.1, C50.1, C51.1, C52.1, C53.1, C54.1, C55.1, C56.1, C57.1, C58.1, C59.1, C60.1, C61.1, C62.1, H2.10, H2.13, H2.18, H2.21, H2.22, H2.29, H2.30, H2.31, H2.47, H2.48, IC1.GND, IC10.GND, IC7.DCDC_GND, IC7.NGND_KEL0, IC7.TEST_MODE, IC7.VSS_1, IC7.VSS_2, IC7.VSS_3, IC7.VSS_4, IC7.VSS_5, IC7.VSS_6, IC7.VSS_7, IC7.VSS_8, IC8.EP, IC9.VSSQ_1, IC9.VSSQ_2, IC9.VSSQ_3, IC9.VSSQ_4, IC9.VSS_1, IC9.VSS_2, IC9.VSS_3, J1.10, J1.11, J1.12, J1.13, J1.14, J1.15, J1.16, J1.VSS, J2.1, J2.14, J2.7, PS1.2, R10.2, R2.1, R26.2, Y1.NC_1, Y1.NC_2; no longer BT1.-, C1.2, C14.2, C15.2, C16.2, C17.2, C18.2, C19.2, C2.2, C20.2, C21.2, C22.2, C23.2, C24.2, C25.2, C26.2, C27.2, C28.2, C29.2, C3.2, C30.2, C31.2, C32.2, C33.2, C34.2, C35.2, C36.2, C37.2, C38.2, C39.2, C40.2, C41.2, C42.2, C43.2, C44.2, C45.2, C46.2, C47.2, C48.2, C49.2, C5.2, C50.2, C51.2, C52.2, C53.2, C54.2, C55.2, C56.2, C57.2, C58.2, C60.2, C61.2, C62.2, C65.2, C66.2, C67.2, C68.2, C69.2, C70.2, C71.2, C72.2, C73.2, C74.2, C76.2, C77.2, C78.2, C79.2, C80.2, C81.2, C82.2, C83.2, C85.2, C86.2, C87.2, C88.2, C89.2, C90.2, C91.2, C92.2, C93.2, C94.2, C95.2, C96.2, D10.1, D5.CATHODE, D8.1, D9.1, FB2.1, IC1.VSSQ_1, IC1.VSSQ_2, IC1.VSSQ_3, IC1.VSSQ_4, IC1.VSS_1, IC1.VSS_2, IC1.VSS_3, IC2.PSC, IC2.PSC#, IC2.VSS, IC2.VSSQ_1, IC2.VSSQ_2, IC3.DIR, IC3.GND, IC4.GND, IC5.DCDC_GND_1, IC5.DCDC_GND_2, IC5.NGND_KEL0, IC5.TEST_MODE, IC5.VDD_SOC_IN_6, IC5.VSS_1, IC5.VSS_2, IC7.GND, J1.7, J2.5, J3.7, J4.7, J5.7, J7.10, J7.8, J7.9, J8.4, J8.5, J9.14, J9.17, J9.21, J9.22, J9.29, J9.30, J9.32, J9.47, J9.48, J9.9, JP1.10, JP1.12, JP1.14, JP1.16, JP1.18, JP1.20, JP1.4, JP1.6, JP1.8, Q1.2, Q1.4, R100.1, R12.1, R14.1, R26.1, R46.1, R64.1, R80.2, R88.1, R91.1, R94.1, R97.1, S1.COM_1, S1.N.O._1, U10.GND, U10.SOC, U11.GND, U11.SOC, U12.GND, U12.SOC, U13.GND, U2.GND, U3.!I2C!/SPI, U3.1_RSVD_GND, U3.2_RSVD_GND, U3.3_RSVD_GND, U3.4_RSVD_GND, U3.5_RSVD_GND, U3.6_RSVD_GND, U3.7_RSVD_GND, U3.8_RSVD_GND, U3.9_RSVD_GND, U3.GND1, U3.GND2, U3.GND3, U3.GND4, U4.EXP, U4.VSS, U4.VSSA, U5.GND, U6.GND, U7.!I2C!/SPI, U7.1_RSVD_GND, U7.2_RSVD_GND, U7.3_RSVD_GND, U7.4_RSVD_GND, U7.5_RSVD_GND, U7.6_RSVD_GND, U7.7_RSVD_GND, U7.8_RSVD_GND, U7.9_RSVD_GND, U7.GND1, U7.GND2, U7.GND3, U7.GND4, U8.GND, U9.!I2C!/SPI, U9.1_RSVD_GND, U9.2_RSVD_GND, U9.3_RSVD_GND, U9.4_RSVD_GND, U9.5_RSVD_GND, U9.6_RSVD_GND, U9.7_RSVD_GND, U9.8_RSVD_GND, U9.9_RSVD_GND, U9.GND1, U9.GND2, U9.GND3, U9.GND4
- net I2C1_SCL: now also H1.44, IC7.GPIO_AD_B1_14; no longer J6.49, R30.1, R41.1, R58.1, R8.2, U12.SCL/SPI_SCK, U13.SCL, U9.SCL/SCLK
- net I2C1_SDA: now also H1.42, IC7.GPIO_AD_B1_15; no longer J6.51, R29.2, R35.1, R59.1, R9.2, U12.SDA/SPI_SDI, U13.SDA, U9.SDA/MOSI/SPI_DATA
- net I2C2_SCL: now also H1.37, IC7.GPIO_AD_B1_08; no longer IC5.GPIO_B0_04, R28.1, R32.1, U10.SCL/SPI_SCK, U3.SCL/SCLK
- net I2C2_SDA: now also H1.35, IC7.GPIO_AD_B1_09; no longer IC5.GPIO_B0_05, R19.2, R31.1, U10.SDA/SPI_SDI, U3.SDA/MOSI/SPI_DATA
- net I2C3_SCL: now also H1.51, IC7.GPIO_AD_B0_08; no longer IC5.GPIO_SD_B0_00, J8.9, R11.1, R34.1, U11.SCL/SPI_SCK, U7.SCL/SCLK
- net I2C3_SDA: now also H1.49, IC7.GPIO_AD_B0_09; no longer IC5.GPIO_SD_B0_01, J8.10, R10.2, R33.1, U11.SDA/SPI_SDI, U7.SDA/MOSI/SPI_DATA
- net JTAG_DE: now also J2.6; no longer JP1.17
- net JTAG_MOD: now also IC7.GPIO_AD_B0_02, R2.2; no longer IC5.GPIO_AD_B0_08, R46.2, TP6.TP
- net JTAG_NTRST: now also IC7.GPIO_AD_B0_05, J2.9, R63.2; no longer IC5.GPIO_AD_B0_11, JP1.3
- net JTAG_RTCK: now also J2.11; no longer JP1.11
- net JTAG_TCK: now also IC7.GPIO_AD_B0_01, J2.4; no longer IC5.GPIO_AD_B0_07, JP1.9, R48.2
- net JTAG_TDI: now also IC7.GPIO_AD_B0_03, J2.3; no longer IC5.GPIO_AD_B0_09, JP1.5, R50.2
- net JTAG_TDO: now also IC7.GPIO_AD_B0_04, J2.5; no longer IC5.GPIO_AD_B0_10, JP1.13
- net JTAG_TMS: now also IC7.GPIO_AD_B0_00, J2.10; no longer IC5.GPIO_AD_B0_06, JP1.7, R47.2
- net N$1: now also IC1.!RESET, R8.1; no longer D4.ANODE, R96.1
- net N$10: now also J1.CMD, R55.2; no longer IC5.GPIO_AD_B0_00, R37.1, R38.2
- net N$11: now also IC9.NC_3, R38.1; no longer C53.1, IC5.XTALO, Q1.1
- net N$13: now also IC8.EN, R60.2; no longer IC1.CLK, R13.2
- net N$2: now also IC9.DQ0, R33.1; no longer C16.1, C17.1, IC5.VDD_HIGH_CAP
- net N$26: now also J1.DAT1, R58.2; no longer IC2.DQ2, R16.1
- net N$3: now also IC1.VDD, R9.2; no longer C20.1, IC5.VDD_SNVS_CAP
- net N$30: now also IC9.DQ7, R12.2; no longer U13.X2, Y1.2
- net N$32: now also IC9.NC_10, R13.2; no longer IC2.RWDS, R21.2
- net N$33: now also IC9.DQ6, R14.2; no longer IC2.DQ1, R23.1
- net N$35: now also IC9.NC_9, R15.2; no longer IC2.DQ0, R24.1
- net N$36: now also IC7.DCDC_LP, L2.2; no longer IC2.DQ3, R25.1
- net N$38: now also J2.2, R27.1; no longer JP1.1, JP1.2, R27.2
- net N$4: now also J1.DATA2, R53.2; no longer C35.1, IC5.DCDC_PSWITCH, R6.1
- net N$41: now also C44.2, IC7.DCDC_PSWITCH, R11.1; no longer U13.X1, Y1.1
- net N$44: now also IC9.NC_8, R17.2; no longer BT1.+, U13.VBAT
- net N$45: now also IC9.DQ4, R18.2; no longer C75.2, U10.SETC
- net N$47: now also IC9.NC_7, R19.2; no longer C59.2, U11.SETC
- net N$5: now also IC9.NC_1, R34.1; no longer C21.1, D6.K, IC5.VDD_SNVS_IN
- net N$50: now also IC9.DQM, R20.2; no longer C84.1, U12.SETP
- net N$51: now also IC9.CLK, R21.2; no longer C58.1, U11.C1
- net N$52: now also IC9.CKE, R22.2; no longer C74.1, U10.C1
- net N$59: now also C20.2, D1.K, IC7.VDD_SNVS_IN; no longer R97.2, U8.ILIM
- net N$6: now also IC9.DQ1, R35.1; no longer IC5.DCDC_LP_1, IC5.DCDC_LP_2, L2.1
- net N$7: now also J1.CD/DAT3, R54.2; no longer C33.1, C34.1, IC5.NVCC_PLL
- net N$8: now also IC9.NC_2, R36.1; no longer IC2.RSTO#, R17.2
- net N$9: now also IC9.DQ2, R37.1; no longer IC5.GPANAIO, TP1.TP
- net NVCC_GPIO_3V3: now also C53.2, C54.2, C55.2, C56.2, C57.2, C58.2, C59.2, C60.2, C61.2, C62.2, C63.2, C64.2, IC7.NVCC_GPIO_1, IC7.NVCC_GPIO_2, IC7.NVCC_GPIO_3, IC7.NVCC_GPIO_4, IC7.NVCC_GPIO_5, IC7.NVCC_GPIO_6, IC7.NVCC_GPIO_7, R62.1; no longer C45.1, C46.1, C47.1, C48.1, IC5.NVCC_GPIO_1, IC5.NVCC_GPIO_2, IC5.NVCC_GPIO_3, R36.2, R37.2, R63.1
- net POR_B: now also C36.2, D4.K, IC7.POR_B, R8.2; no longer IC5.POR_B, R40.2
- net RTC_XTALO: now also C42.2, IC7.RTC_XTALO, Y2.OUT/IN; no longer C64.2, IC5.RTC_XTALO, Q3.1
- net SDRAM_3V3: now also FB1.2, IC9.VDDQ_1, IC9.VDDQ_2, IC9.VDDQ_3, IC9.VDDQ_4, IC9.VDD_1, IC9.VDD_2, IC9.VDD_3; no longer C5.1, IC1.VDDQ_1, IC1.VDDQ_2, IC1.VDDQ_3, IC1.VDDQ_4, IC1.VDD_1, IC1.VDD_2, IC1.VDD_3, L1.2, R15.2
- net SEMC_A0: now also IC7.GPIO_EMC_16, R49.2; no longer IC1.A0, IC5.GPIO_EMC_09
- net SEMC_A1: now also IC7.GPIO_EMC_17, R50.2; no longer IC1.A1, IC5.GPIO_EMC_10
- net SEMC_A10: now also IC7.GPIO_EMC_15, R48.2; no longer IC1.A10, IC5.GPIO_EMC_23
- net SEMC_A11: now also IC7.GPIO_EMC_26, R24.1; no longer IC1.A11, IC5.GPIO_EMC_19
- net SEMC_A12: now also IC7.GPIO_EMC_27, R23.1; no longer IC1.A12, IC5.GPIO_EMC_20
- net SEMC_A2: now also IC7.GPIO_EMC_18, R51.2; no longer IC1.A2, IC5.GPIO_EMC_11
- net SEMC_A3: now also IC7.GPIO_EMC_19, R52.2; no longer IC1.A3, IC5.GPIO_EMC_12
- net SEMC_A4: now also IC7.GPIO_EMC_20, R32.1; no longer IC1.A4, IC5.GPIO_EMC_13
- net SEMC_A5: now also IC7.GPIO_EMC_21, R31.1; no longer IC1.A5, IC5.GPIO_EMC_14
- net SEMC_A6: now also IC7.GPIO_EMC_22, R30.1; no longer IC1.A6, IC5.GPIO_EMC_15
- net SEMC_A7: now also IC7.GPIO_EMC_23, R29.1; no longer IC1.A7, IC5.GPIO_EMC_16
- net SEMC_A8: now also IC7.GPIO_EMC_24, R28.1; no longer IC1.A8, IC5.GPIO_EMC_17
- net SEMC_A9: now also IC7.GPIO_EMC_25, R25.1; no longer IC1.A9, IC5.GPIO_EMC_18
- net SEMC_BA0: now also IC7.GPIO_EMC_13, R46.2; no longer IC1.BA0, IC5.GPIO_EMC_21
- net SEMC_BA1: now also IC7.GPIO_EMC_14, R47.2; no longer IC1.BA1, IC5.GPIO_EMC_22
- net SEMC_CAS: now also IC7.GPIO_EMC_10, R43.2; no longer IC1.!CAS, IC5.GPIO_EMC_24
- net SEMC_CKE: now also IC7.GPIO_EMC_29, R22.1; no longer IC1.CKE, IC5.GPIO_EMC_27, R14.2
- net SEMC_CLK: now also IC7.GPIO_EMC_30, R21.1; no longer IC5.GPIO_EMC_26, R13.1
- net SEMC_CS0: now also IC7.GPIO_EMC_12, R45.2; no longer IC1.!CS, IC5.GPIO_EMC_29, R15.1
- net SEMC_D0: now also IC7.GPIO_EMC_00, R33.2; no longer IC1.DQ0, IC5.GPIO_EMC_00
- net SEMC_D1: now also IC7.GPIO_EMC_01, R34.2; no longer IC1.DQ1, IC5.GPIO_EMC_01
- net SEMC_D10: now also IC7.GPIO_EMC_34, R17.1; no longer IC1.DQ10, IC5.GPIO_EMC_32
- net SEMC_D11: now also IC7.GPIO_EMC_35, R16.1; no longer IC1.DQ11, IC5.GPIO_EMC_33
- net SEMC_D12: now also IC7.GPIO_EMC_36, R15.1; no longer IC1.DQ12, IC5.GPIO_EMC_34
- net SEMC_D13: now also IC7.GPIO_EMC_37, R14.1; no longer IC1.DQ13, IC5.GPIO_EMC_35
- net SEMC_D14: now also IC7.GPIO_EMC_38, R13.1; no longer IC1.DQ14, IC5.GPIO_EMC_36
- net SEMC_D15: now also IC7.GPIO_EMC_39, R12.1; no longer IC1.DQ15, IC5.GPIO_EMC_37
- net SEMC_D2: now also IC7.GPIO_EMC_02, R35.2; no longer IC1.DQ2, IC5.GPIO_EMC_02
- net SEMC_D3: now also IC7.GPIO_EMC_03, R36.2; no longer IC1.DQ3, IC5.GPIO_EMC_03
- net SEMC_D4: now also IC7.GPIO_EMC_04, R37.2; no longer IC1.DQ4, IC5.GPIO_EMC_04
- net SEMC_D5: now also IC7.GPIO_EMC_05, R38.2; no longer IC1.DQ5, IC5.GPIO_EMC_05
- net SEMC_D6: now also IC7.GPIO_EMC_06, R39.2; no longer IC1.DQ6, IC5.GPIO_EMC_06
- net SEMC_D7: now also IC7.GPIO_EMC_07, R40.2; no longer IC1.DQ7, IC5.GPIO_EMC_07
- net SEMC_D8: now also IC7.GPIO_EMC_32, R19.1; no longer IC1.DQ8, IC5.GPIO_EMC_30
- net SEMC_D9: now also IC7.GPIO_EMC_33, R18.1; no longer IC1.DQ9, IC5.GPIO_EMC_31
- net SEMC_DM0: now also IC7.GPIO_EMC_08, R41.2; no longer IC1.DQML, IC5.GPIO_EMC_08
- net SEMC_DM1: now also IC7.GPIO_EMC_31, R20.1; no longer IC1.DQMH, IC5.GPIO_EMC_38
- net SEMC_RAS: now also IC7.GPIO_EMC_11, R44.2; no longer IC1.!RAS, IC5.GPIO_EMC_25
- net SEMC_WE: now also IC7.GPIO_EMC_09, R42.2; no longer IC1.!WE, IC5.GPIO_EMC_28
- net SPI1_MISO: now also H1.18, IC7.GPIO_AD_B0_13; no longer IC5.GPIO_AD_B0_02, J1.4, J3.4, J4.4, J5.4
- net SPI1_MOSI: now also H1.16, IC7.GPIO_AD_B0_12; no longer J1.3, J3.3, J4.3, J5.3, R39.1
- net SPI1_SCK: now also H1.12, IC7.GPIO_AD_B0_10; no longer J1.5, J3.5, J4.5, J5.5, R38.1
- net UART3_RX: now also H1.52, IC7.GPIO_AD_B0_15; no longer IC5.GPIO_AD_B1_07, J7.5
- net UART3_TX: now also H1.50, IC7.GPIO_AD_B0_14; no longer IC5.GPIO_AD_B1_06, J7.3
- net USER_LED: now also R63.1; no longer R50.1
- net VDD_USB_3V: now also C14.2, C4.2, IC7.VDD_USB_CAP; no longer C43.1, C44.1, IC5.VDD_USB_CAP
- net XTALI: now also C39.2, IC7.XTALI, R10.1, Y1.XTAL_2; no longer C54.1, IC5.XTALI, Q1.3, R12.2
Other:
- note added: "DETECTION PIN NOT NEEDED"
- note removed: "DO NOT USE"
- note removed: "Gyroscopes"
- note removed: "Magnetometers"
- note removed: "PU/PD LOGIC: SERIAL INTERFACE IS ALWAYS RESET WHEN USB PORT IS DISCONNECTED"
- note removed: "Pin not connected"
- note removed: "Pin not connected."
