File: projects/onboard_flight_computer/obc.brd (EAGLE design)
At the start: 90.2 x 95.9 mm, 191 parts, among them IC1 IS42S16160J-6BLI, IC2 S26KS512SDPBHI020, IC3 74LVC2T45GS,115, IC4 74LVCH1T45GS,132, IC5 MIMXRT1052DVJ6B, IC7 74LVCH1T45GS,132, IC8 74LVCH1T45GS,132, J1 504050-0791, J2 DX4R205JJAR1800, J3 504050-0791, J4 504050-0791, J5 504050-0791, J6 ESQ-126-37-G-D, J7 FH28-10S-0.5SH_05_, J8 504050-1091, J9 ESQ-126-37-G-D, Q1 FA-128, Q3 FC-12M, U10 HONEYWELL_HMC5983-TRHONEYWELL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, U11 HONEYWELL_HMC5983-TRHONEYWELL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, U12 HONEYWELL_HMC5983-TRHONEYWELL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, U13 DS1307N, U2 MCP1702T-1802E/CB, U3 NXP_FXAS21002CQR1NXP_FXAS2100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, U4 MK20DX128VFM5, U5 NLX2G14CMUTCG, U6 NTSX2102GU8H, U7 NXP_FXAS21002CQR1NXP_FXAS2100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, U8 NX5P3090UKZ, U9 NXP_FXAS21002CQR1NXP_FXAS2100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, Y1 ECS-.327-12.5-13X

Commit message: Update obc.brd
Parts:
- removed BT1: BA2032SM, BA2032SM:BAT_BA2032SM
- removed C65, C69, C82: 10 uF, rcl:C0402K
- removed C66: 2.2 uF, rcl:C0402K
- removed C67, C72, C73, C76, C77, C78, C81, C85, C88, C89, C92, C93, C96: 0.1 uF, rcl:C0402K
- removed C68, C86, C90, C94: 1.0 uF, rcl:C0402K
- removed C70, C71: 22 pF, rcl:C0402K
- removed C74, C80, C83: 4.7 uF, rcl:C0402K
- removed C75, C84: 0.22 uF, rcl:C0402K
- removed C79: 1000 pF, rcl:C0402K
- removed C87, C91, C95: 100 nF, rcl:C0402K
- removed D10, D8, D9: 0402ESDA-MLP1, 0402ESDA-MLP1:DIONC1105X44N
- removed D5: KINGBRIGHT_KPT-1608SGCKINGBRIGHT_KPT-1608SGC_0_0, Kingbright - KPT-1608SGC:KINGBRIGHT_KPT-1608SGC_0
- removed D6: RB521S30T1G, RB521S30T1G:SODFL1608X70N
- removed FB2: MPZ1608S331A, MPZ1608S331A:BEADC1608X95N
- removed IC2: S26KS512SDPBHI020, SDRAM_and_HyperFlash:BGA24C100P5X5_600X800X100
- removed IC3: 74LVC2T45GS,115, 74LVC2T45GS_115:74AXP2T3407GSX
- removed IC4: 74LVCH1T45GS,132, 74LVCH1T45GS_132:74LVC1G3157GS132
- removed IC5: MIMXRT1052DVJ6B, MIMXRT1052DVJ6B:BGA196C80P14X14_1200X1200X161
- removed J3, J4, J5: 504050-0791, 504050-0791:504050-0791
- removed J6, J9: ESQ-126-37-G-D, ESQ-126-37-G-D:ESQ-126-Y-X
- removed J7: FH28-10S-0.5SH_05_, FH28-10S-0.5SH_05_:FH2810S05SH05
- removed J8: 504050-1091, 504050-1091:504050-1091
- removed JP1: 20, pinhead:2X10
- removed L1: 120 Ohm, inductors:0402
- removed Q1: FA-128, crystal:FA-128
- removed Q3: FC-12M, crystal:FC-12M
- removed R114, R134: 1k Ohm, rcl:R0402
- removed R80: CSTCE8M00G55-R0, CSTCE8M00G55-R0:CSTCE12M0G55-R0
- removed S1: TL3301AF260QG, TL3301AF260QG:TL3301AF260QG
- removed TP1, TP10, TP12, TP13, TP14, TP15, TP3: TPTP06R, testpad:TP06R
- removed U10, U11, U12: HONEYWELL_HMC5983-TRHONEYWELL_HMC5983-TR_0_0, Honeywell - HMC5983-TR:HONEYWELL_HMC5983-TR_0
- removed U13: DS1307N, DS1307N:DIP762W47P254L991H457Q8
- removed U2: MCP1702T-1802E/CB, MCP1702T1802ECB:SOT-23A_MC
- removed U3, U7, U9: NXP_FXAS21002CQR1NXP_FXAS21002CQR1_0_0, NXP - FXAS21002CQR1:NXP_FXAS21002CQR1_0
- removed U4: MK20DX128VFM5, MK20DX128VFM5:QFN50P500X500X100-33N
- removed U5: NLX2G14CMUTCG, NLX2G14CMUTCG:UDFN6_1X1
- removed U6: NTSX2102GU8H, NTSX2102GU8H:QFN40P140X120X50-8N
- removed U8: NX5P3090UKZ, NX5P3090UKZ:BGA12CP40_3X4_135X165X56B26N
- added C4: 0.1uF, rcl:C0402K
- added D1, D3: BAT54XV2T1G, BAT54XV2T1G:SODFL1608X70N
- added H1, H2: ESQ-126-39-G-D, ESQ-126-39-G-D:SAMTEC_ESQ-126-39-G-D
- added IC10: IS25LP064A-JBLE, IS25LP064A-JBLE:SOIC127P790X216-8N
- added IC9: IS42S16160J-6TL, IS42S16160J-6TL:SOP80P1176X120-54N
- added PS1: PJ-040D, PJ-040D:PJ040D
- added R10: 2.2M Ohm, rcl:R0402
- added R11: 30k Ohm, rcl:R0402
- added R19, R28, R29, R30, R31, R32, R33, R34, R35, R41, R42, R45, R49, R51, R52, R53, R54, R55, R56, R57, R60, R61, R62: 0 Ohm, rcl:R0402
- added TP5, TP8: TPTP06R, testpad:TP06R
- added Y2: ECS-.327-7-12-TR, ECS-.327-7-12-TR:ECS327712TR
- C14: value 0.22uF -> 10 uF
- C16, C19, C31, C33, C48: value 4.7uF -> 0.22uF
- C17, C23, C36: value 0.22uF -> 0.1uF
- C18, C24, C35: value 0.22uF -> 4.7uF
- C2, C51: value 0.1uF -> 4.7uF
- C3: value 4.7uF -> 1.0 uF
- C32, C43: value 10uF -> 0.1uF
- C37: value 33uF -> 0.1uF
- C39: value 4.7uF -> 4.7pF
- C40: value 0.22uF -> 4.7pF
- C41, C42: value 0.22uF -> 10pF
- C44, C45, C46, C47: value 0.1uF -> 0.22uF
- C5: value 22uF -> 1.0uF
- C50: value 0.1uF -> 1.0uF
- C52: value 4.7uF -> 1.0uF
- C53, C54, C55: value 4.7uF -> 0.1uF
- C57: value 0.1 uF -> 0.1uF
- C58: value 4.7 uF -> 0.1uF
- C59: value 0.22 uF -> 0.1uF
- C60, C61, C62: value 0.1 uF -> 4.7uF
- C63, C64: value 18pF -> 4.7uF
- D2: value RB521S30T1G -> BAT54XV2T1G; device RB521S30T1G:SODFL1608X70N -> BAT54XV2T1G:SODFL1608X70N
- D4: value KINGBRIGHT_KPT-1608SGCKINGBRIGHT_KPT-1608SGC_0_0 -> BAT54XV2T1G; device Kingbright - KPT-1608SGC:KINGBRIGHT_KPT-1608SGC_0 -> BAT54XV2T1G:SODFL1608X70N
- FB1: value MPZ1608S331A -> BLM15AG121SN1D; device MPZ1608S331A:BEADC1608X95N -> BLM15AG121SN1D:NFZ15SG152SN10B
- IC1: value IS42S16160J-6BLI -> TPS3839L30DBZR; device SDRAM_and_HyperFlash:BGA54C80P9X9_800X800X120 -> TPS3839L30DBZR:SOT95P237X112-3N
- IC7: value 74LVCH1T45GS,132 -> MIMXRT1021DAG5A; device 74LVCH1T45GS_132:74LVC1G3157GS132 -> MIMXRT1021DAG5A:QFP50P2200X2200X160-144N
- IC8: value 74LVCH1T45GS,132 -> MIC94305YMT-TR; device 74LVCH1T45GS_132:74LVC1G3157GS132 -> MIC94305YMT-TR:SON50P160X120X60-5N
- J1: value 504050-0791 -> 504077-1891; device 504050-0791:504050-0791 -> 504077-1891:5040771891
- J2: value DX4R205JJAR1800 -> 12214-8250-00FR; device DX4R205JJAR1800:JAE_DX4R205JJAR1800 -> 12214-8250-00FR:12214825000FR
- L2: value 4.7 uH -> SRN4026-4R7M; device inductors:0402 -> SRN4026-4R7M:SRN4026
- R1, R5, R59: value 0 Ohm -> 10k Ohm
- R12: value 2.2M Ohm -> 0 Ohm
- R14, R15: value 100K Ohm -> 0 Ohm
- R17, R18, R3: value 10k Ohm -> 0 Ohm
- R26: value 10k Ohm -> 100 Ohm
- R36, R37: value 4.7K Ohm -> 0 Ohm
- R46: value 10K Ohm -> 0 Ohm
- R6: value 30K Ohm -> 10k Ohm
- R8: value 4.7 k -> 0 Ohm; device rcl:R0805 -> rcl:R0402
- R9: value 4.7k -> 1k Ohm; device rcl:R0805 -> rcl:R0402
- Y1: value ECS-.327-12.5-13X -> XRCGB24M000F2P01R0; device ECS-.327-12.5-13X:XTAL_ECS-.327-12.5-13X -> XRCGB24M000F2P01R0:XRCGB24M000F2P01R0
- moved C16 80.8 mm to (9.83, 38.4)
- moved C36 73.0 mm to (64.7, 23.7), turned to 180 degrees
- moved C39 72.8 mm to (59.9, 18.7)
- moved C53 72.8 mm to (7.24, 22.0), turned to 90 degrees
- moved C54 72.4 mm to (9.45, 22.0), turned to 90 degrees
- moved C17 71.9 mm to (11.4, 38.4), turned to 270 degrees
- moved C55 71.9 mm to (11.4, 22.0), turned to 90 degrees
- moved C24 68.8 mm to (55.7, 22.8), turned to 90 degrees
- moved FB1 68.6 mm to (19.9, 54.9), turned to 180 degrees
- moved R9 68.0 mm to (67.5, 24.2), turned to 0 degrees
- moved C6 67.3 mm to (40.5, 67.5)
- moved C11 66.9 mm to (43.8, 67.5), turned to 90 degrees
- moved C51 66.8 mm to (16.0, 27.9)
- moved IC8 66.8 mm to (74.7, 28.7), turned to 90 degrees
- moved J1 66.1 mm to (72.0, 14.8), turned to 270 degrees
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Connections:
- removed net 12V_BUS: J9.23, J9.24
- removed net 12V_PDM1: J9.8
- removed net 12V_PDM2: J9.10
- removed net 3V3_PDM10: J9.20
- removed net 3V3_PDM8: J9.18
- removed net 3V3_PDM9: C57.1, C60.1, C61.1, C62.1, C72.1, C73.1, C85.1, C86.1, C88.1, C89.1, C90.1, C92.1, C93.1, C94.1, C96.1, J7.6, J9.19, U10.13, U10.2, U10.4, U10.6, U11.13, U11.2, U11.4, U11.6, U12.13, U12.2, U12.4, U12.6, U3.13, U3.15, U3.17, U3.18, U7.13, U7.15, U7.17, U7.18, U9.13, U9.15, U9.17, U9.18
- removed net 5V_BUS: J9.25, J9.26, R8.1, R9.1, U13.8
- removed net 5V_PDM5: J8.3, J9.13
- removed net 5V_PDM6: J1.1, J3.1, J4.1, J5.1, J9.15
- removed net 5V_PDM7: J8.1, J9.16
- removed net 5V_USB_CHARGE: D8.2, FB1.1, J2.1, J6.32
- removed net AAA: U8.A1
- removed net BATV_BUS: J9.45, J9.46
- removed net BATV_PDM3: J9.11
- removed net BATV_PDM4: J9.12
- removed net CAN_STBY: IC5.G14, R44.2
- removed net CHASSIS: J7.7, J9.50
- removed net DCDC_3V3: C1.1, C14.1, C15.1, C18.1, C19.1, C2.1, C3.1, D6.2, IC5.E6, IC5.F5, IC5.N14, IC5.P12, L1.1, R1.2, R114.2, R134.2, R27.1, R63.2, R7.2
- removed net FLASH_RST: IC5.D7, R2.1
- removed net FLASH_VCC: C51.1, C52.1, C55.1, C56.1, IC2.B4, IC2.D1, IC2.E4, IC5.K5, R17.1, R18.1, R3.1, R4.2
- removed net FLEXSPI_CLK_B: IC2.B1, IC5.P2
- removed net FLEXSPI_D0_B: IC2.D5, IC5.M4
- removed net FLEXSPI_D1_B: IC2.E3, IC5.M3
- removed net FLEXSPI_D2_B: IC2.E2, IC5.M5
- removed net FLEXSPI_D3_B: IC2.E1, IC5.L5
- removed net FLEXSPI_DQS: IC5.N3, R21.1
- removed net GPIO_AD_B1_00: IC5.J11, R58.2
- removed net GPIO_AD_B1_01: IC5.K11, R59.2
- removed net LDO_1V8: C49.1, C50.1, R4.1, TP3.TP, U2.2
- removed net MCU_DCDC_IN: C39.1, C40.1, C41.1, C42.1, IC5.K4, IC5.L1, IC5.L2, R6.2, R7.1
- removed net N$27: IC2.A5, R18.2
- removed net N$29: IC2.A4, R2.2
- removed net N$31: IC2.C2, R20.2, R3.2
- removed net N$34: IC2.B2, R22.2
- removed net N$37: JP1.19, R26.2
- removed net N$39: D2.1, JP1.15
- removed net N$40: C32.1, C38.1, R1.1, U2.3
- removed net N$46: C75.1, U10.8
- removed net N$48: C59.1, U11.8
- removed net N$49: C84.2, U12.12
- removed net N$53: C63.2, IC5.N9, Q3.2
- removed net N$54: U6.5
- removed net N$56: C83.1, U12.10
- removed net N$57: TP12.TP, U6.3
- removed net N$60: TP13.TP, U6.6
- removed net N$67: C91.1, U7.16
- removed net N$71: C87.1, U3.16
- removed net N$72: C95.1, U9.16
- removed net N$76: D11.2, R134.1
- removed net P3V3_SDA: C67.1, C68.1, C69.1, C76.1, C78.1, IC3.1, IC4.1, IC7.1, IC8.1, U4.1, U4.11, U4.7, U5.5, U6.1
- removed net P5V_SDA: C65.1, C81.1, C82.1, FB1.2, U4.6, U8.B1, U8.B2, U8.C1
- removed net P5V_SDA_S: C80.1, U8.C2, U8.D1, U8.D2
- removed net PCM_IN: J9.35, J9.36
- removed net POWER_EN: U4.31
- removed net POWER_LED: D5.2, R114.1
- removed net SDA_EXTAL: C70.1, R80.3, U4.17
- removed net SDA_LED: D4.1, U4.29
- removed net SDA_RST: TP7.TP, U4.19
- removed net SDA_RST_TGTMCU_B: C79.1, R40.1, S1.2, S1.4, U4.21, U6.2, U6.7
- removed net SDA_RX_EN: IC4.5
- removed net SDA_SPI0_CS: TP15.TP, U4.23
- removed net SDA_SPI0_RST_B: TP14.TP, U4.22
- removed net SDA_SPI0_SCK: IC8.3, U4.26
- removed net SDA_SPI0_SIN: IC3.3, U4.28
- removed net SDA_SPI0_SOUT: IC7.3, U4.27
- removed net SDA_SWD_EN: IC8.5, U5.6
- removed net SDA_SWD_EN_B: U4.16, U5.1
- removed net SDA_SWD_OE: IC7.5, U5.4
- removed net SDA_SWD_OE_B: U4.20, U5.3
- removed net SDA_USBSHIELD: FB2.2, J2.S4, J2.S5
- removed net SDA_USB_CONN_DN: D10.2, J2.2
- removed net SDA_USB_CONN_DP: D9.2, J2.3
- removed net SDA_USB_DN: U4.4
- removed net SDA_USB_DP: U4.3
- removed net SDA_VOUT33: C66.1, U4.5
- removed net SDA_XTAL: C71.1, R80.1, U4.18
- removed net SPI1_EN_1: IC5.A9, J1.2
- removed net SPI1_EN_2: IC5.B9, J3.2
- removed net SPI1_EN_3: IC5.C9, J4.2
- removed net SPI1_EN_4: IC5.D9, J5.2
- removed net SPI1_NSS_1: J1.6, R43.1
- removed net SPI1_NSS_2: IC5.F11, J3.6
- removed net SPI1_NSS_3: J4.6, R44.1
- removed net SPI1_NSS_4: IC5.H14, J5.6
- removed net SWD_CLK: IC8.4, R48.1
- removed net SWD_DIO: IC3.6, IC7.4, R47.1
- removed net TC_SDA_USB_ID_TP: J2.4, TP10.TP
- removed net UART1_RXD: IC4.4, IC5.L14
- removed net UART1_RX_TGTMCU_R: IC4.3, U4.25
- removed net UART1_TXD: IC3.7, IC5.K14
- removed net UART1_TX_TGTMCU_R: IC3.2, U4.24
- removed net UART2_RX: IC5.M12, J6.3
- removed net UART2_TX: IC5.L11, J6.1
- removed net UART8_RX: IC5.J13, J8.8
- removed net UART8_TX: IC5.L13, J8.7
- removed net USB_OTG1_ID: IC5.H10, R36.1, R39.2
- removed net USB_OTG1_OC: IC5.G11, R43.2
- removed net VDD_SOC_IN: C22.1, C23.1, C24.1, C25.1, C26.1, C27.1, C28.1, C29.1, C30.1, C31.1, IC5.F6, IC5.F7, IC5.F8, IC5.F9, IC5.J5, R5.1
- removed net VTRG_FAULT_B: U4.32, U8.A2
- removed net V_TGTMCU: C77.1, IC3.8, IC4.6, IC7.6, IC8.6, U6.8
- new net 5V_USB_OTG: C3.2, IC7.59
- new net FLASH_3V3: C32.2, C5.2, IC10.8, R1.1, R4.2
- new net GPANAIO: IC7.71, TP7.TP
- new net GPIO_EMC_16: IC9.23, R49.1
- new net GPIO_EMC_17: IC9.24, R50.1
- new net GPIO_EMC_18: IC9.25, R51.1
- new net GPIO_EMC_19: IC9.26, R52.1
- new net GPIO_EMC_20: IC9.29, R32.2
- new net GPIO_EMC_21: IC9.30, R31.2
- new net GPIO_EMC_22: IC9.31, R30.2
- new net GPIO_EMC_23: IC9.32, R29.2
- new net GPIO_EMC_24: IC9.33, R28.2
- new net GPIO_EMC_25: IC9.34, R25.2
- new net GPIO_EMC_26: IC9.35, R24.2
- new net GPIO_EMC_27: IC9.36, R23.2
- new net INT1_COMBO: IC7.27, R7.1
- new net JTAG_DACK: J2.13, R26.1
- new net JTAG_NSRST: D2.1, J2.12
- new net N$12: IC9.11, R39.1
- new net N$14: IC9.13, R40.1
- new net N$15: J1.5, R56.2
- new net N$16: IC9.15, R41.1
- new net N$17: IC9.16, R42.1
- new net N$18: IC9.17, R43.1
- new net N$19: IC9.18, R44.1
- new net N$20: IC9.19, R45.1
- new net N$21: IC9.20, R46.1
- new net N$22: IC9.21, R47.1
- new net N$23: IC9.22, R48.1
- new net N$24: D3.2, D4.2, R60.1, R61.1
- new net N$25: J1.7, R57.2
- new net N$42: IC9.47, R16.2
- new net NVCC_PLL: C22.2, IC7.72
- new net NVCC_SD0: C1.2, C2.2, IC7.44, R3.2
- new net PMIC_STBY_REQ: IC7.54, TP6.TP
- new net RTC_XTALI: C41.2, IC7.57, Y2.1
- new net SD1_CLK: IC7.45, R56.1
- new net SD1_CMD: IC7.46, R5.2, R55.1
- new net SD1_D0: IC7.43, R57.1, R6.2
- new net SD1_D1: IC7.42, R58.1
- new net SD1_D2: IC7.48, R53.1
- new net SD1_D3: IC7.47, R54.1
- new net SD_CD_SW: IC7.41, J1.9, R59.1
- new net SD_PWREN: D3.1, R7.2
- new net SPI1_EN0: H1.9, IC7.92
- new net SPI1_EN1: H1.10, IC7.91
- new net SPI1_EN2: H1.22, IC7.90
- new net SPI1_EN3: H1.21, IC7.89
- new net SPI1_PCS0: H1.7, IC7.97
- new net SPI1_PCS1: H1.8, IC7.88
- new net SPI1_PCS2: H1.20, IC7.87
- new net SPI1_PCS3: H1.19, IC7.84
- new net UART1_RX: H1.4, IC7.101
- new net UART1_TX: H1.2, IC7.105
- new net UART4_RX: H1.3, IC7.79
- new net UART4_TX: H1.1, IC7.80
- new net USB_OTG1_CHD: IC7.66, TP5.TP
- new net VDD_HIGH_CAP: C23.2, C24.2, IC7.65
- new net VDD_SNVS_CAP: C21.2, IC7.56
- new net VSD_3V3: C38.2, C49.2, C52.2, IC8.3, J1.4
- new net WAKEUP: IC7.52, TP8.TP
- new net XTALO: C40.2, IC7.68, Y1.1
- net 3V3_BUS: now also C15.2, C16.2, C17.2, C18.2, C19.2, C37.2, C43.2, C47.2, C48.2, C50.2, C51.2, D1.2, D11.2, FB1.1, H2.27, H2.28, IC7.34, IC7.38, IC7.69, IC7.73, IC8.4, J2.8, R11.2, R27.2, R3.1, R4.1, R5.1, R59.2, R6.1, R61.2, R62.2, R9.1; no longer IC5.J6, J9.27, J9.28
- net ANT_BURN_WIRE1: now also H1.23, IC7.83; no longer IC5.A10, J6.24
- net ANT_BURN_WIRE2: now also H1.25, IC7.78; no longer IC5.D10, J6.26
- net BCR_OUT: now also H2.41, H2.42, H2.43, H2.44, PS1.1; no longer J9.41, J9.42, J9.43, J9.44
- net DCDC_OUT: now also C25.2, C26.2, C27.2, C28.2, C29.2, C30.2, C31.2, C33.2, C34.2, C35.2, C45.2, C46.2, IC7.102, IC7.114, IC7.134, IC7.31, IC7.39, IC7.5, IC7.86, L2.1; no longer C36.1, C37.1, L2.2, R5.2
- net DTR: now also H1.5, IC7.26; no longer IC5.C10, J8.6
- net FLEXSPI_CLK: now also IC10.6, IC7.24; no longer IC5.L4, R22.1
- net FLEXSPI_D0_A: now also IC10.5, IC7.23; no longer IC5.P3, R24.2
- net FLEXSPI_D1_A: now also IC10.2, IC7.21; no longer IC5.N4, R23.2
- net FLEXSPI_D2_A: now also IC10.3, IC7.22; no longer IC5.P4, R16.2
- net FLEXSPI_D3_A: now also IC10.7, IC7.25; no longer IC5.P5, R25.2
- net FLEXSPI_SS0: now also IC10.1, IC7.19, R1.2; no longer IC5.L3, R20.1
- net GND: now also C1.1, C14.1, C15.1, C16.1, C17.1, C18.1, C19.1, C2.1, C20.1, C21.1, C22.1, C23.1, C24.1, C25.1, C26.1, C27.1, C28.1, C29.1, C3.1, C30.1, C31.1, C32.1, C33.1, C34.1, C35.1, C36.1, C37.1, C38.1, C39.1, C4.1, C40.1, C41.1, C42.1, C43.1, C44.1, C45.1, C46.1, C47.1, C48.1, C49.1, C5.1, C50.1, C51.1, C52.1, C53.1, C54.1, C55.1, C56.1, C57.1, C58.1, C59.1, C60.1, C61.1, C62.1, H2.10, H2.13, H2.18, H2.21, H2.22, H2.29, H2.30, H2.31, H2.47, H2.48, IC1.1, IC10.4, IC7.103, IC7.113, IC7.135, IC7.35, IC7.40, IC7.51, IC7.6, IC7.60, IC7.64, IC7.70, IC7.85, IC8.5, IC9.12, IC9.28, IC9.41, IC9.46, IC9.52, IC9.54, IC9.6, J1.10, J1.11, J1.12, J1.13, J1.14, J1.15, J1.16, J1.6, J2.1, J2.14, J2.7, PS1.2, R10.2, R2.1, R26.2, Y1.2, Y1.4; no longer BT1.-, C1.2, C14.2, C15.2, C16.2, C17.2, C18.2, C19.2, C2.2, C20.2, C21.2, C22.2, C23.2, C24.2, C25.2, C26.2, C27.2, C28.2, C29.2, C3.2, C30.2, C31.2, C32.2, C33.2, C34.2, C35.2, C36.2, C37.2, C38.2, C39.2, C40.2, C41.2, C42.2, C43.2, C44.2, C45.2, C46.2, C47.2, C48.2, C49.2, C5.2, C50.2, C51.2, C52.2, C53.2, C54.2, C55.2, C56.2, C57.2, C58.2, C60.2, C61.2, C62.2, C65.2, C66.2, C67.2, C68.2, C69.2, C70.2, C71.2, C72.2, C73.2, C74.2, C76.2, C77.2, C78.2, C79.2, C80.2, C81.2, C82.2, C83.2, C85.2, C86.2, C87.2, C88.2, C89.2, C90.2, C91.2, C92.2, C93.2, C94.2, C95.2, C96.2, D10.1, D5.1, D8.1, D9.1, FB2.1, IC1.A1, IC1.A3, IC1.B7, IC1.C3, IC1.D7, IC1.E3, IC1.J1, IC2.B3, IC2.B5, IC2.C1, IC2.C5, IC2.E5, IC3.4, IC3.5, IC4.2, IC5.A1, IC5.A14, IC5.G9, IC5.K6, IC5.K9, IC5.N1, IC5.N2, IC7.2, J1.7, J2.5, J3.7, J4.7, J5.7, J7.10, J7.8, J7.9, J8.4, J8.5, J9.14, J9.17, J9.21, J9.22, J9.29, J9.30, J9.32, J9.47, J9.48, J9.9, JP1.10, JP1.12, JP1.14, JP1.16, JP1.18, JP1.20, JP1.4, JP1.6, JP1.8, Q1.2, Q1.4, R12.1, R14.1, R26.1, R46.1, R80.2, S1.1, S1.3, U10.11, U10.9, U11.11, U11.9, U12.11, U12.9, U13.4, U2.1, U3.1, U3.10, U3.14, U3.19, U3.20, U3.21, U3.22, U3.23, U3.24, U3.5, U3.6, U3.7, U3.8, U3.9, U4.2, U4.33, U4.8, U5.2, U6.4, U7.1, U7.10, U7.14, U7.19, U7.20, U7.21, U7.22, U7.23, U7.24, U7.5, U7.6, U7.7, U7.8, U7.9, U8.B3, U8.C3, U8.D3, U9.1, U9.10, U9.14, U9.19, U9.20, U9.21, U9.22, U9.23, U9.24, U9.5, U9.6, U9.7, U9.8, U9.9
- net I2C1_SCL: now also H1.44, IC7.75; no longer J6.49, R58.1, R8.2, U12.1, U13.6, U9.11
- net I2C1_SDA: now also H1.42, IC7.74; no longer J6.51, R59.1, R9.2, U12.16, U13.5, U9.12
- net I2C2_SCL: now also H1.37, IC7.82; no longer IC5.C8, U10.1, U3.11
- net I2C2_SDA: now also H1.35, IC7.81; no longer IC5.B8, U10.16, U3.12
- net I2C3_SCL: now also H1.51, IC7.100; no longer IC5.J4, J8.9, U11.1, U7.11
- net I2C3_SDA: now also H1.49, IC7.99; no longer IC5.J3, J8.10, U11.16, U7.12
- net JTAG_DE: now also J2.6; no longer JP1.17
- net JTAG_MOD: now also IC7.109, R2.2; no longer IC5.F13, R46.2, TP6.TP
- net JTAG_NTRST: now also IC7.106, J2.9, R63.2; no longer IC5.G10, JP1.3
- net JTAG_RTCK: now also J2.11; no longer JP1.11
- net JTAG_TCK: now also IC7.110, J2.4; no longer IC5.F12, JP1.9, R48.2
- net JTAG_TDI: now also IC7.108, J2.3; no longer IC5.F14, JP1.5, R50.2
- net JTAG_TDO: now also IC7.107, J2.5; no longer IC5.G13, JP1.13
- net JTAG_TMS: now also IC7.111, J2.10; no longer IC5.E14, JP1.7, R47.2
- net N$1: now also IC1.2, R8.1; no longer D4.2
- net N$10: now also J1.3, R55.2; no longer IC5.M14, R37.1, R38.2
- net N$11: now also IC9.10, R38.1; no longer C53.1, IC5.N11, Q1.1
- net N$13: now also IC8.1, R60.2; no longer IC1.F2, R13.2
- net N$2: now also IC9.2, R33.1; no longer C16.1, C17.1, IC5.P8
- net N$26: now also J1.8, R58.2; no longer IC2.C4, R16.1
- net N$3: now also IC1.3, R9.2; no longer C20.1, IC5.M10
- net N$30: now also IC9.53, R12.2; no longer U13.2, Y1.2
- net N$32: now also IC9.51, R13.2; no longer IC2.C3, R21.2
- net N$33: now also IC9.50, R14.2; no longer IC2.D2, R23.1
- net N$35: now also IC9.48, R15.2; no longer IC2.D3, R24.1
- net N$36: now also IC7.36, L2.2; no longer IC2.D4, R25.1
- net N$38: now also J2.2, R27.1; no longer JP1.1, JP1.2, R27.2
- net N$4: now also J1.1, R53.2; no longer C35.1, IC5.K3, R6.1
- net N$41: now also C44.2, IC7.37, R11.1; no longer U13.1, Y1.1
- net N$44: now also IC9.45, R17.2; no longer BT1.+, U13.3
- net N$45: now also IC9.44, R18.2; no longer C75.2, U10.12
- net N$47: now also IC9.42, R19.2; no longer C59.2, U11.12
- net N$5: now also IC9.4, R34.1; no longer C21.1, D6.1, IC5.M9
- net N$50: now also IC9.39, R20.2; no longer C84.1, U12.8
- net N$51: now also IC9.38, R21.2; no longer C58.1, U11.10
- net N$52: now also IC9.37, R22.2; no longer C74.1, U10.10
- net N$59: now also C20.2, D1.1, IC7.55; no longer U8.A3
- net N$6: now also IC9.5, R35.1; no longer IC5.M1, IC5.M2, L2.1
- net N$7: now also J1.2, R54.2; no longer C33.1, C34.1, IC5.P10
- net N$8: now also IC9.7, R36.1; no longer IC2.A2, R17.2
- net N$9: now also IC9.8, R37.1; no longer IC5.N10, TP1.TP
- net NVCC_GPIO_3V3: now also C53.2, C54.2, C55.2, C56.2, C57.2, C58.2, C59.2, C60.2, C61.2, C62.2, C63.2, C64.2, IC7.104, IC7.11, IC7.112, IC7.144, IC7.20, IC7.29, IC7.77, R62.1; no longer C45.1, C46.1, C47.1, C48.1, IC5.E9, IC5.F10, IC5.J10, R36.2, R37.2, R63.1
- net POR_B: now also C36.2, D4.1, IC7.50, R8.2; no longer IC5.M7, R40.2
- net RTC_XTALO: now also C42.2, IC7.58, Y2.2; no longer C64.2, IC5.P9, Q3.1
- net SDRAM_3V3: now also FB1.2, IC9.1, IC9.14, IC9.27, IC9.3, IC9.43, IC9.49, IC9.9; no longer C5.1, IC1.A7, IC1.A9, IC1.B3, IC1.C7, IC1.D3, IC1.E7, IC1.J9, L1.2, R15.2
- net SEMC_A0: now also IC7.142, R49.2; no longer IC1.H7, IC5.C2
- net SEMC_A1: now also IC7.141, R50.2; no longer IC1.H8, IC5.G1
- net SEMC_A10: now also IC7.143, R48.2; no longer IC1.H9, IC5.G2
- net SEMC_A11: now also IC7.130, R24.1; no longer IC1.G2, IC5.B4
- net SEMC_A12: now also IC7.129, R23.1; no longer IC1.G1, IC5.A3
- net SEMC_A2: now also IC7.140, R51.2; no longer IC1.J8, IC5.G3
- net SEMC_A3: now also IC7.139, R52.2; no longer IC1.J7, IC5.H1
- net SEMC_A4: now also IC7.138, R32.1; no longer IC1.J3, IC5.A6
- net SEMC_A5: now also IC7.137, R31.1; no longer IC1.J2, IC5.B6
- net SEMC_A6: now also IC7.136, R30.1; no longer IC1.H3, IC5.B1
- net SEMC_A7: now also IC7.133, R29.1; no longer IC1.H2, IC5.A5
- net SEMC_A8: now also IC7.132, R28.1; no longer IC1.H1, IC5.A4
- net SEMC_A9: now also IC7.131, R25.1; no longer IC1.G3, IC5.B2
- net SEMC_BA0: now also IC7.2, R46.2; no longer IC1.G7, IC5.C1
- net SEMC_BA1: now also IC7.1, R47.2; no longer IC1.G8, IC5.F1
- net SEMC_CAS: now also IC7.7, R43.2; no longer IC1.F7, IC5.D3
- net SEMC_CKE: now also IC7.127, R22.1; no longer IC1.F3, IC5.A2, R14.2
- net SEMC_CLK: now also IC7.126, R21.1; no longer IC5.B3, R13.1
- net SEMC_CS0: now also IC7.3, R45.2; no longer IC1.G9, IC5.E1, R15.1
- net SEMC_D0: now also IC7.18, R33.2; no longer IC1.A8, IC5.E3
- net SEMC_D1: now also IC7.17, R34.2; no longer IC1.B9, IC5.F3
- net SEMC_D10: now also IC7.122, R17.1; no longer IC1.D1, IC5.D5
- net SEMC_D11: now also IC7.121, R16.1; no longer IC1.C2, IC5.C4
- net SEMC_D12: now also IC7.120, R15.1; no longer IC1.C1, IC5.D4
- net SEMC_D13: now also IC7.119, R14.1; no longer IC1.B2, IC5.E5
- net SEMC_D14: now also IC7.118, R13.1; no longer IC1.B1, IC5.C3
- net SEMC_D15: now also IC7.117, R12.1; no longer IC1.A2, IC5.E4
- net SEMC_D2: now also IC7.16, R35.2; no longer IC1.B8, IC5.F4
- net SEMC_D3: now also IC7.15, R36.2; no longer IC1.C9, IC5.G4
- net SEMC_D4: now also IC7.14, R37.2; no longer IC1.C8, IC5.F2
- net SEMC_D5: now also IC7.13, R38.2; no longer IC1.D9, IC5.G5
- net SEMC_D6: now also IC7.12, R39.2; no longer IC1.D8, IC5.H5
- net SEMC_D7: now also IC7.10, R40.2; no longer IC1.E9, IC5.H4
- net SEMC_D8: now also IC7.124, R19.1; no longer IC1.E1, IC5.C6
- net SEMC_D9: now also IC7.123, R18.1; no longer IC1.D2, IC5.C5
- net SEMC_DM0: now also IC7.9, R41.2; no longer IC1.E8, IC5.H3
- net SEMC_DM1: now also IC7.125, R20.1; no longer IC1.F1, IC5.D6
- net SEMC_RAS: now also IC7.4, R44.2; no longer IC1.F8, IC5.D2
- net SEMC_WE: now also IC7.8, R42.2; no longer IC1.F9, IC5.D1
- net SPI1_MISO: now also H1.18, IC7.95; no longer IC5.M11, J1.4, J3.4, J4.4, J5.4
- net SPI1_MOSI: now also H1.16, IC7.96; no longer J1.3, J3.3, J4.3, J5.3, R39.1
- net SPI1_SCK: now also H1.12, IC7.98; no longer J1.5, J3.5, J4.5, J5.5, R38.1
- net UART3_RX: now also H1.52, IC7.93; no longer IC5.K10, J7.5
- net UART3_TX: now also H1.50, IC7.94; no longer IC5.J12, J7.3
- net USER_LED: now also R63.1; no longer R50.1
- net VDD_USB_3V: now also C14.2, C4.2, IC7.61; no longer C43.1, C44.1, IC5.K8
- net XTALI: now also C39.2, IC7.67, R10.1, Y1.3; no longer C54.1, IC5.P11, Q1.3, R12.2
Routing:
- net GND: track 829.9 -> 236.1 mm, vias 25 -> 57
- net 3V3_BUS: track 62.3 -> 486.1 mm, vias 3 -> 17
- net 3V3_PDM9: track 341.1 -> 0.00 mm, vias 8 -> 0
- net DCDC_3V3: track 285.2 -> 0.00 mm, vias 10 -> 0
- net FLASH_VCC: track 228.5 -> 0.00 mm, vias 7 -> 0
- net P3V3_SDA: track 206.9 -> 0.00 mm, vias 10 -> 0
- net N$40: track 179.3 -> 0.00 mm, vias 4 -> 0
- net VDD_SOC_IN: track 177.4 -> 0.00 mm, vias 11 -> 0
- net 5V_PDM6: track 171.9 -> 0.00 mm, vias 5 -> 0
- net XTALI: track 151.3 -> 14.2 mm, vias 5 -> 0
- net MCU_DCDC_IN: track 131.1 -> 0.00 mm, vias 7 -> 0
- net N$11: track 162.2 -> 36.0 mm, vias 2 -> 0
- net SDA_RST_TGTMCU_B: track 122.6 -> 0.00 mm, vias 5 -> 0
- net P5V_SDA: track 117.6 -> 0.00 mm, vias 8 -> 0
- net JTAG_TMS: track 142.8 -> 28.8 mm, vias 3 -> 2
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