File: REALcontrol_boardv18.brd (EAGLE design)
At the start: 95.9 x 90.2 mm, 35 parts, among them IC3 4050D, IC4 LP298XS, X2 MICROSD

Commit message: Add files via upload
Parts:
- moved X2 4.03 mm to (39.8, 53.8)
- moved U$2 3.48 mm to (31.9, 29.1)
Routing:
- net 5V_2: track 127.1 -> 138.5 mm
- net RX: track 35.3 -> 44.7 mm
- net N$24: track 57.5 -> 64.1 mm
- net N$6: track 112.6 -> 118.8 mm
- net N$23: track 40.9 -> 46.7 mm
- net N$27: track 50.5 -> 55.3 mm
- net N$5: track 108.9 -> 113.4 mm
- net N$26: track 41.2 -> 45.3 mm
- net +3V3: track 68.6 -> 72.6 mm
- net DO: track 50.7 -> 53.9 mm
- net VCC: track 110.3 -> 108.9 mm
- net TX: track 36.8 -> 36.3 mm
- net N$3: track 36.0 -> 36.6 mm
